File: hw/sch_pcb/PIND01.kicad_pcb (KiCad board)
At the start: 2 copper layers, 40.1 x 40.1 mm, 34 parts, among them J1 JUMP_2x1, J2 JUMP_2x1, J3 JUMP_2x1, J4 JUMP_2x1, M1 HOLE, M2 HOLE, M3 HOLE, M4 HOLE

Commit message: Update Project to KiCADv7.
Other:
- net class Default removed
